Commit message: tested + camera bugged

File: mrvk_description/urdf/common.urdf.xacro (robot description, xacro)
@@ -1,14 +1,14 @@
 <?xml version="1.0"?>
 <robot name="kv01" xmlns:xacro="http://www.ros.org/wiki/xacro">
-  <macro name = "inertia_zaklad">
+  <xacro:macro name = "inertia_zaklad">
     <inertia ixx="0.1" ixy="0.0" ixz="0.0" iyy="0.1" iyz="0.0" izz="0.1"/>
-  </macro>
-  <macro name = "inertia_motor">
+  </xacro:macro>
+  <xacro:macro name = "inertia_motor">
     <inertia ixx="1" ixy="0.0" ixz="0.0" iyy="1" iyz="0.0" izz="1"/>
-  </macro>
-  <macro name="dynamika">
+  </xacro:macro>
+  <xacro:macro name="dynamika">
     <dynamics fricction = "1" damping ="1"/>
-  </macro>
-<macro name="gazebo_def_part" params="part material">
+  </xacro:macro>
+<xacro:macro name="gazebo_def_part" params="part material">
   <gazebo reference="${part}">
     <mu1>0.5</mu1>
@@ -17,6 +17,6 @@
     <material>Gazebo/${material}</material>
   </gazebo>
-</macro>
-<macro name="klb_vlastnosti" params="meno">
+</xacro:macro>
+<xacro:macro name="klb_vlastnosti" params="meno">
   <gadzebo reference="${meno}">
     <erp>0.1</erp>
@@ -26,12 +26,12 @@
     <implicitSpringDamper>true</implicitSpringDamper>
   </gadzebo>
-</macro>
-<macro name="klb_def" params="meno">
+</xacro:macro>
+<xacro:macro name="klb_def" params="meno">
   <gadzebo reference="${meno}">
   </gadzebo>
-</macro>
+</xacro:macro>
 <!--parametre-->
-  <property name="M_PI" value="3.14159"/>
-  <property name="WHEEL_RADIUS" value="0.115"/>
-  <property name="ODOMETRY_CONSTANT" value="0.006546076617684" />
+  <xacro:property name="M_PI" value="3.14159"/>
+  <xacro:property name="WHEEL_RADIUS" value="0.115"/>
+  <xacro:property name="ODOMETRY_CONSTANT" value="0.006546076617684" />
 </robot>

File: mrvk_description/urdf/mrvk.urdf.xacro (robot description, xacro)
@@ -16,5 +16,5 @@
   <xacro:macro name="mrvk_base" params="parent *origin end_point">
     <joint name="footprint_to_base" type="fixed">
-      <insert_block name="origin" />
+      <xacro:insert_block name="origin" />
       <parent link="${parent}"/>
       <child link="base_link"/>
@@ -326,5 +326,5 @@
     </joint>
     <actuator name="camera_horizontal_motor">
-      <hardwareInterface>PositionJointInterface</hardwareInterface>
+      <hardwareInterface>hardware_interface/PositionJointInterface</hardwareInterface>
       <mechanicalReduction>1</mechanicalReduction>
     </actuator>
@@ -336,5 +336,5 @@
     </joint>
     <actuator name="camera_vertical_motor">
-      <hardwareInterface>PositionJointInterface</hardwareInterface>
+      <hardwareInterface>hardware_interface/PositionJointInterface</hardwareInterface>
       <mechanicalReduction>1</mechanicalReduction>
     </actuator>
