Commit message: navigation basic setup

File: mrvk_description/urdf/mrvk.urdf.xacro (robot description, xacro)
@@ -15,9 +15,9 @@
        name="mrvk" >
   <xacro:macro name="mrvk_base" params="parent *origin end_point">
-    <joint name="footprint_to_base" type="fixed">
+    <!--joint name="footprint_to_base" type="fixed">
       <xacro:insert_block name="origin" />
       <parent link="${parent}"/>
       <child link="base_link"/>
-    </joint>
+    </joint-->
     <link name="base_link"/>
    <joint name="base_to_stabilizer" type="fixed">

File: mrvk_description/urdf/robot.urdf.xacro (robot description, xacro)
@@ -20,5 +20,5 @@
   <xacro:include filename="$(find mrvk_description)/urdf/kv01.urdf.xacro" />
   <!-- Used for fixing robot to Gazebo -->
-  <link name="world"/>
+  <!--link name="world"/-->
   <!-- arm -->
   <xacro:mrvk_base parent="world" end_point = "base_end_point">

Commit message: recovered source from robot, added vision - kinect, pavement

File: mrvk_description/urdf/mrvk.urdf.xacro (robot description, xacro)
@@ -85,5 +85,5 @@
 	  <origin xyz="-0.03 0 0.0375"/>
 	  <axis xyz="0 0 1"/>
-	  <limit effort="30.0" lower="-2.09439" upper="${M_PI}" velocity="0.5"/>
+	  <limit effort="30.0" lower="-2.09439" upper="${M_PI}" velocity="5"/>
   </joint>
   <link name="camera_l">
@@ -134,5 +134,5 @@
     </link>
     <joint name="camera_r_to_camera" type="revolute">
-      <limit effort="30.0" lower="-0.523598" upper="${M_PI/2}" velocity="0.5"/>
+      <limit effort="30.0" lower="-0.523598" upper="${M_PI/2}" velocity="5"/>
       <parent link="camera_r"/>
       <child link="camera"/>

Commit message: kinect config updated

File: mrvk_description/urdf/mrvk.urdf.xacro (robot description, xacro)
@@ -163,5 +163,5 @@
           <parent link="veza"/>
           <child link="kinect_ir"/>
-          <origin rpy="1.57 0 1.57" xyz="0.0 -0.070 0.158"/>
+          <origin rpy="0 0 -1.57" xyz="0.0 -0.070 0.158"/>
       </joint>
     <link name="wheel_frame_l">

Commit message: utm odometry node fix, costmap common config update, xacro gps frame added

File: mrvk_description/urdf/mrvk.urdf.xacro (robot description, xacro)
@@ -324,4 +324,16 @@
     </joint>
     <link name="${end_point}"/>
+    <joint name="base_to_gps" type="fixed">
+      <parent link="base_link"/>
+      <child link="gps"/>
+      <origin rpy="0 0 0" xyz="0 0 2"/>
+    </joint>
+    <link name="gps"/>
+<joint name="gps_to_vo" type="fixed">
+      <parent link="gps"/>
+      <child link="vo"/>
+      <origin rpy="0 0 0" xyz="0 0 0"/>
+    </joint>
+    <link name="vo"/>
   <transmission name="mrvk_left_transmission">
     <type>transmission_interface/SimpleTransmission</type>

Commit message: kinect position updated

File: mrvk_description/urdf/mrvk.urdf.xacro (robot description, xacro)
@@ -154,14 +154,14 @@
       </link>
       <joint name="kinect_to_veza" type="fixed">
-          <parent link="veza"/>
+          <parent link="base_stabilized"/>
           <child link="kinect"/>
-          <origin rpy=" 0 0 0" xyz="0 0 0.150"/>
+          <origin rpy=" 0 0 0" xyz="0.100 0 0.509"/>
       </joint>
       <link name="kinect_ir">
       </link>
       <joint name="kinect_ir_to_veza" type="fixed">
-          <parent link="veza"/>
+          <parent link="kinect"/>
           <child link="kinect_ir"/>
-          <origin rpy="0 0 -1.57" xyz="0.0 -0.070 0.158"/>
+          <origin rpy="1.57 0 1.57" xyz="0.0 -0.070 0"/>
       </joint>
     <link name="wheel_frame_l">

File: mrvk_description/urdf/robot.urdf.xacro (robot description, xacro)
@@ -18,5 +18,5 @@
   <xacro:include filename="$(find mrvk_description)/urdf/common.urdf.xacro" />
   <xacro:include filename="$(find mrvk_description)/urdf/mrvk.urdf.xacro" />
-  <xacro:include filename="$(find mrvk_description)/urdf/kv01.urdf.xacro" />
+ <!--  <xacro:include filename="$(find mrvk_description)/urdf/kv01.urdf.xacro" /> -->
   <!-- Used for fixing robot to Gazebo -->
   <!--link name="world"/-->
@@ -25,5 +25,5 @@
      <origin xyz="0 0 0.13" rpy="0 0 0" />
   </xacro:mrvk_base>
-  <xacro:kv01_arm parent="base_end_point" end_point = "tool_point">
-  </xacro:kv01_arm>
+  <!--<xacro:kv01_arm parent="base_end_point" end_point = "tool_point">-->
+  <!--</xacro:kv01_arm>-->
 </robot>

Commit message: data update

File: mrvk_description/urdf/mrvk.urdf.xacro (robot description, xacro)
@@ -14,355 +14,367 @@
        xmlns:physics="http://playerstage.sourceforge.net/gazebo/xmlschema/#physics"
        name="mrvk" >
-  <xacro:macro name="mrvk_base" params="parent *origin end_point">
-    <!--joint name="footprint_to_base" type="fixed">
-      <xacro:insert_block name="origin" />
-      <parent link="${parent}"/>
-      <child link="base_link"/>
-    </joint-->
-    <link name="base_link"/>
-   <joint name="base_to_stabilizer" type="fixed">
-      <origin xyz="0 0 0"/>
-      <parent link="base_link"/>
-      <child link="base_stabilized"/>
-    </joint>
-<!--todo narazniky -->
-    <link name="base_stabilized">
-      <visual>
-	<geometry>
-        <box size="0.47 .315 .168"/>
-	</geometry>
-	<origin xyz="0 0 0"/>
-	<material name="Blue"/>
-      </visual>
-      <inertial>
-	<mass value="10"/>
-	<inertia_zaklad/>
-      </inertial>
-      <collision>
-	<geometry>
-	<box size="0.5 .31 .30"/>
-	</geometry>
-	<origin xyz="0 0 0.08"/>
-     </collision>
-   </link>
-  <joint name="stabilizer_to_imu" type="fixed">
-    <origin xyz="-0.1 0.1 -0.01"/>
-    <parent link="base_stabilized"/>
-    <child link="imu"/>
-  </joint>
-  <link name = "imu"/>
-  <link name="laser">
-    <visual>
-      <geometry>
-	  <cylinder length="0.03" radius="0.025"/>
-      </geometry>
-      <material name="Black"/>
-    </visual>
-      <inertial>
-	<mass value="0.1"/>
-	<xacro:inertia_zaklad/>
-      </inertial>
-    </link>
-    <joint name="base_to_scan" type="fixed">
-    <parent link="base_stabilized"/>
-    <child link="laser"/>
-    <origin xyz="0.181 0 0.099"/>
-    </joint>
-    <link name="veza">
-    <visual>
-      <geometry>
-	<cylinder length="0.045" radius="0.0665"/>
-      </geometry>
-      <material name="White"/>
-    </visual>
-    <inertial>
-	<mass value="0.3"/>
-	<inertia_zaklad/>
-      </inertial>
-    </link>
-    <joint name="scan_to_veza" type="revolute"><!--todo premenovat na base_to_veza-->
-      <parent link="base_stabilized"/>
-	<child link="veza"/>
-	  <origin xyz="0.14 0 0.136"/>
-	  <axis xyz="0 0 1"/>
-	  <limit effort="30.0" lower="-2.09439" upper="${M_PI}" velocity="5"/>
-  </joint>
-  <link name="camera_l">
-      <visual>
-	<geometry>
-	  <box size="0.07 .03 .08"/>
-	</geometry>
-      <material name="Black"/>
-      </visual>
-      <inertial>
-	<mass value="0.1"/>
-	<inertia_zaklad/>
-      </inertial>
-    </link>
-    <joint name="veza_to_camera_l" type="fixed">
-      <parent link="veza"/>
-      <child link="camera_l"/>
-      <origin xyz="0 0.05 0.0575"/>
-    </joint>
-    <link name="camera_r">
-      <visual>
-	<geometry>
-	  <box size="0.07 .03 .08"/>
-	</geometry>
-	<material name="Black"/>
-      </visual>
-      <inertial>
-	<mass value="0.1"/>
-	<inertia_zaklad/>
-      </inertial>
-    </link>
-    <joint name="veza_to_camera_r" type="fixed">
-      <parent link="veza"/>
-      <child link="camera_r"/>
-      <origin xyz="0 -0.05 0.0575"/>
-    </joint>
-    <link name="camera">
-      <visual>
-	<geometry>
-	  <box size="0.075 .06 .06"/>
-	</geometry>
-      <material name="Black"/>
-      </visual>
-      <inertial>
-	<mass value="0.4"/>
-	<inertia_zaklad/>
-      </inertial>
-    </link>
-    <joint name="camera_r_to_camera" type="revolute">
-      <limit effort="30.0" lower="-0.523598" upper="${M_PI/2}" velocity="5"/>
-      <parent link="camera_r"/>
-      <child link="camera"/>
-      <origin rpy=" ${M_PI/2} 0 0" xyz="0 0.05 0.01"/>
-      <axis xyz="0 0 1"/>
-    </joint>
-      <link name="kinect">
-          <visual>
-              <geometry>
-                  <box size=" .065 0.25 .075"/>
-              </geometry>
-              <material name="kinect"/>
-          </visual>
-          <inertial>
-              <mass value="1.5"/>
-              <inertia_zaklad/>
-          </inertial>
-      </link>
-      <joint name="kinect_to_veza" type="fixed">
-          <parent link="veza"/>
-          <child link="kinect"/>
-          <origin rpy=" 0 0 0" xyz="0 0 0.150"/>
-      </joint>
-      <link name="kinect_ir">
-      </link>
-      <joint name="kinect_ir_to_veza" type="fixed">
-          <parent link="veza"/>
-          <child link="kinect_ir"/>
-          <origin rpy="0 0 -1.57" xyz="0.0 -0.070 0.158"/>
-      </joint>
-    <link name="wheel_frame_l">
-      <visual>
-      <geometry>
-	<box size="0.4 .025 .1"/>
-      </geometry>
-	<material name="White"/>
-      </visual>
-      <inertial>
-	<mass value="1.3"/>
-	<inertia_zaklad/>
-      </inertial>
-    </link>
-    <joint name="wheel_joint_left" type="continuous">
-	<!--limit rychlosti v impulzoch za 10ms-->
-      <limit effort="30.0" velocity="${1000*ODOMETRY_CONSTANT}"/>
-      <parent link="wheel_frame_l"/>
-      <child link="wheel_frame_l_rotation"/>
-      <origin rpy="${-M_PI/2} 0 0"/>
-      <axis xyz="0 0 1"/>
-    </joint>
-    <link name="wheel_frame_l_rotation">
-    </link>
-    <joint name="base_link_to_wheel_frame_l" type="fixed">
-      <parent link="base_stabilized"/>
-	<child link="wheel_frame_l"/>
-	<origin xyz="0 +0.1775 -0.05"/>
-	<axis xyz="0 1 0"/>
-    </joint>
-    <link name="wheel_frame_r">
-      <visual>
-	<geometry>
-	  <box size="0.4 .025 .1"/>
-	</geometry>
-	<material name="White"/>
-      </visual>
-      <inertial>
-	<mass value="1.3"/>
-	<inertia_zaklad/>
-      </inertial>
-    </link>
-    <joint name="wheel_joint_right" type="continuous">
-	<!--limit rychlosti v impulzoch za 10ms-->
-      <limit effort="30.0" velocity="${1000*ODOMETRY_CONSTANT}"/>
-      <parent link="wheel_frame_r"/>
-      <child link="wheel_frame_r_rotation"/>
-      <origin rpy="${M_PI/2} 0 0"/>
-      <axis xyz="0 0 -1"/>
-    </joint>
-    <link name="wheel_frame_r_rotation">
-    </link>
-    <joint name="base_link_to_wheel_frame_r" type="fixed">
-      <parent link="base_stabilized"/>
-      <child link="wheel_frame_r"/>
-      <origin xyz="0 -0.1775 -0.05"/>
-      <axis xyz="0 1 0"/>
-    </joint>
-    <link name="wheel_lp">
-      <visual>
-	<geometry>
-	  <cylinder radius="${WHEEL_RADIUS}" length="0.065"/>
-	</geometry>
-      <material name="Black"/>
-      </visual>
-      <inertial>
-	<mass value="0.5"/>
-	<inertia_zaklad/>
-      </inertial>
-      <collision>
-	  <geometry>
-	    <cylinder radius="${WHEEL_RADIUS}" length="0.065"/>
-	  </geometry>
-      </collision>
-    </link>
-    <joint name="wheel_frame_l_to_wheel_lp" type="continuous">
-       <parent link="wheel_frame_l"/>
-       <child link="wheel_lp"/>
-       <origin rpy=" ${M_PI/2} 0 0" xyz="0.145 0.05 -0.01"/>
-       <axis xyz="0 0 1"/>
-       <mimic joint= "wheel_joint_left" multiplier="-1" />
-    </joint>
-    <link name="wheel_lz">
-      <visual>
-      <geometry>
-	<cylinder radius="${WHEEL_RADIUS}" length="0.065"/>
-      </geometry>
-	<material name="Black"/>
-      </visual>
-      <inertial>
-	<mass value="0.5"/>
-	<inertia_zaklad/>
-      </inertial>
-      <collision>
-	  <geometry>
-	    <cylinder radius="${WHEEL_RADIUS}" length="0.065"/>
-	  </geometry>
-      </collision>
-    </link>
-    <joint name="wheel_frame_l_to_wheel_lz" type="continuous">
-      <parent link="wheel_frame_l"/>
-      <child link="wheel_lz"/>
-      <origin rpy=" ${M_PI/2} 0 0" xyz="-0.145 0.05 -0.01"/>
-      <axis xyz="0 0 1"/>
-      <mimic joint= "wheel_joint_left" multiplier="-1" />
-    </joint>
-    <link name="wheel_pp">
-      <visual>
-	<geometry>
-	  <cylinder radius="${WHEEL_RADIUS}" length="0.065"/>
-	</geometry>
-	<material name="Black"/>
-      </visual>
-      <inertial>
-	<mass value="0.5"/>
-	<inertia_zaklad/>
-      </inertial>
-      <collision>
-	  <geometry>
-	    <cylinder radius="${WHEEL_RADIUS}" length="0.065"/>
-	  </geometry>
-      </collision>
-    </link>
-    <joint name="wheel_frame_r_to_wheel_pp" type="continuous">
-      <parent link="wheel_frame_r"/>
-      <child link="wheel_pp"/>
-      <origin rpy=" ${M_PI/2} 0 0" xyz="0.145 -0.05 -0.01"/>
-      <axis xyz="0 0 1"/>
-      <mimic joint= "wheel_joint_right" multiplier="-1" />
-    </joint>
-    <link name="wheel_pz">
-      <visual>
-      <geometry>
-	<cylinder radius="${WHEEL_RADIUS}" length="0.065"/>
-      </geometry>
-      <material name="Black"/>
-      </visual>
-      <inertial>
-	<mass value="0.5"/>
-	<inertia_zaklad/>
-    </inertial>
-      <collision>
-	  <geometry>
-	    <cylinder radius="${WHEEL_RADIUS}" length="0.065"/>
-	  </geometry>
-      </collision>
-    </link>
-    <joint name="wheel_frame_r_to_wheel_pz" type="continuous">
-      <parent link="wheel_frame_r"/>
-      <child link="wheel_pz"/>
-      <origin rpy=" ${M_PI/2} 0 0" xyz="-0.145 -0.05 -0.01"/>
-      <axis xyz="0 0 1"/>
-      <mimic joint= "wheel_joint_right" multiplier="-1" />
-    </joint>
-    <joint name="end_point_connetion" type="fixed">
-      <parent link="base_stabilized"/>
-      <child link="${end_point}"/>
-      <origin rpy="0 0 0" xyz="0 0 0"/>
-      <axis xyz="0 0 1"/>
-    </joint>
-    <link name="${end_point}"/>
-  <transmission name="mrvk_left_transmission">
-    <type>transmission_interface/SimpleTransmission</type>
-    <joint name="wheel_joint_left">
-      <hardwareInterface>hardware_interface/VelocityJointInterface</hardwareInterface>
-    </joint>
-    <actuator name="mrvk_motor_left">
-			<hardwareInterface>hardware_interface/VelocityJointInterface</hardwareInterface>
-      <mechanicalReduction>${1/ODOMETRY_CONSTANT}</mechanicalReduction>
-    </actuator>
-  </transmission>
-  <transmission name="mrvk_right_transmission">
-    <type>transmission_interface/SimpleTransmission</type>
-    <joint name="wheel_joint_right">
-      <hardwareInterface>hardware_interface/VelocityJointInterface</hardwareInterface>
-    </joint>
-    <actuator name="mrvk_motor_right">
-			<hardwareInterface>hardware_interface/VelocityJointInterface</hardwareInterface>
-      <mechanicalReduction>${1/ODOMETRY_CONSTANT}</mechanicalReduction>
-    </actuator>
-  </transmission>
-<!--${1/ODOMETRY_CONSTANT/WHEEL_RADIUS}-->
-  <transmission name="camera_horizontal_transmission">
-    <type>transmission_interface/SimpleTransmission</type>
-    <joint name="scan_to_veza">
-      <hardwareInterface>hardware_interface/PositionJointInterface</hardwareInterface>
-    </joint>
-    <actuator name="camera_horizontal_motor">
-      <hardwareInterface>hardware_interface/PositionJointInterface</hardwareInterface>
-      <mechanicalReduction>1</mechanicalReduction>
-    </actuator>
-  </transmission>
-  <transmission name="camera_vertical_transmission">
-    <type>transmission_interface/SimpleTransmission</type>
-    <joint name="camera_r_to_camera">
-      <hardwareInterface>hardware_interface/PositionJointInterface</hardwareInterface>
-    </joint>
-    <actuator name="camera_vertical_motor">
-      <hardwareInterface>hardware_interface/PositionJointInterface</hardwareInterface>
-      <mechanicalReduction>1</mechanicalReduction>
-    </actuator>
-  </transmission>
+    <xacro:macro name="mrvk_base" params="parent *origin end_point">
+        <joint name="footprint_to_base" type="fixed">
+          <xacro:insert_block name="origin" />
+          <parent link="${parent}"/>
+          <child link="base_link"/>
+        </joint>
+        <link name="base_link"/>
+        <joint name="base_to_stabilizer" type="fixed">
+            <origin xyz="0 0 0"/>
+            <parent link="base_link"/>
+            <child link="base_stabilized"/>
+        </joint>
+        <!--todo narazniky -->
+        <link name="base_stabilized">
+            <visual>
+                <geometry>
+                    <box size="0.47 .315 .168"/>
+                </geometry>
+                <origin xyz="0 0 0"/>
+                <material name="Blue"/>
+            </visual>
+            <inertial>
+                <mass value="10"/>
+                <inertia_zaklad/>
+            </inertial>
+            <collision>
+                <geometry>
+                    <box size="0.5 .31 .30"/>
+                </geometry>
+                <origin xyz="0 0 0.08"/>
+            </collision>
+        </link>
+        <joint name="stabilizer_to_imu" type="fixed">
+            <origin xyz="-0.1 0.1 -0.01"/>
+            <parent link="base_stabilized"/>
+            <child link="imu"/>
+        </joint>
+        <link name = "imu"/>
+        <link name="laser">
+            <visual>
+                <geometry>
+                    <cylinder length="0.03" radius="0.025"/>
+                </geometry>
+                <material name="Black"/>
+            </visual>
+            <inertial>
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
File: mrvk_description/urdf/robot.urdf.xacro (robot description, xacro)
@@ -20,8 +20,8 @@
   <xacro:include filename="$(find mrvk_description)/urdf/kv01.urdf.xacro" />
   <!-- Used for fixing robot to Gazebo -->
-  <!--link name="world"/-->
+  <link name="world"/>
   <!-- arm -->
   <xacro:mrvk_base parent="world" end_point = "base_end_point">
-     <origin xyz="0 0 0.13" rpy="0 0 0" />
+     <origin xyz="0 0 0.174" rpy="0 0 0" />
   </xacro:mrvk_base>
   <xacro:kv01_arm parent="base_end_point" end_point = "tool_point">

Commit message: iai kinect added , kinect position updated

File: mrvk_description/urdf/mrvk.urdf.xacro (robot description, xacro)
@@ -156,5 +156,5 @@
             <parent link="base_stabilized"/>
             <child link="kinect"/>
-            <origin rpy=" 0 0.44 0" xyz="0.100 0 0.509"/>
+            <origin rpy=" 0 0.30 0" xyz="0.100 0 0.509"/>
         </joint>
         <link name="kinect_ir">
@@ -163,5 +163,5 @@
             <parent link="kinect"/>
             <child link="kinect_ir"/>
-            <origin rpy="1.57 0 1.57" xyz="0.0 0 0"/>
+            <origin rpy="1.57 0 1.57" xyz="0.0 -0.070 0"/>
         </joint>
         <link name="wheel_frame_l">

Commit message: kinect position updated

File: mrvk_description/urdf/mrvk.urdf.xacro (robot description, xacro)
@@ -156,5 +156,5 @@
             <parent link="base_stabilized"/>
             <child link="kinect"/>
-            <origin rpy=" 0 0.30 0" xyz="0.100 0 0.509"/>
+            <origin rpy=" 0 0.35 0" xyz="0.100 0 0.489"/>
         </joint>
         <link name="kinect_ir">

Commit message: driver update

File: mrvk_description/urdf/mrvk.urdf.xacro (robot description, xacro)
@@ -15,12 +15,12 @@
        name="mrvk" >
     <xacro:macro name="mrvk_base" params="parent *origin end_point">
-        <joint name="footprint_to_base" type="fixed">
+        <!--joint name="footprint_to_base" type="fixed">
           <xacro:insert_block name="origin" />
           <parent link="${parent}"/>
           <child link="base_link"/>
-        </joint>
+        </joint-->
         <link name="base_link"/>
         <joint name="base_to_stabilizer" type="fixed">
-            <origin xyz="0 0 0"/>
+            <origin xyz="0 0 0" rpy="0 0 1.5707"/>
             <parent link="base_link"/>
             <child link="base_stabilized"/>

Commit message: datasets_from camera

File: mrvk_description/urdf/mrvk.urdf.xacro (robot description, xacro)
@@ -15,12 +15,19 @@
        name="mrvk" >
     <xacro:macro name="mrvk_base" params="parent *origin end_point">
-        <joint name="footprint_to_base" type="fixed">
-          <xacro:insert_block name="origin" />
-          <parent link="${parent}"/>
-          <child link="base_link"/>
-        </joint>
+        <!--<joint name="footprint_to_base" type="fixed">-->
+          <!--<xacro:insert_block name="origin" />-->
+          <!--<parent link="${parent}"/>-->
+          <!--<child link="base_link"/>-->
+        <!--</joint>-->
         <link name="base_link"/>
+        <!--<joint name="fbase_to_stabilizer" type="continuous">-->
+            <!--<limit effort="30.0"  velocity="5"/>-->
+            <!--<origin xyz="0 0 0.174"/>-->
+            <!--<parent link="base_link"/>-->
+            <!--<child link="base_stabilized"/>-->
+            <!--<axis xyz="0 0 1"/>-->
+        <!--</joint>-->
         <joint name="base_to_stabilizer" type="fixed">
-            <origin xyz="0 0 0"/>
+            <origin xyz="0 0 0.174"/>
             <parent link="base_link"/>
             <child link="base_stabilized"/>

File: mrvk_description/urdf/robot.urdf.xacro (robot description, xacro)
@@ -20,8 +20,8 @@
  <!--  <xacro:include filename="$(find mrvk_description)/urdf/kv01.urdf.xacro" /> -->
   <!-- Used for fixing robot to Gazebo -->
-  <link name="world"/>
+  <!--<link name="world"/>-->
   <!-- arm -->
   <xacro:mrvk_base parent="world" end_point = "base_end_point">
-     <origin xyz="0 0 0.174" rpy="0 0 0" />
+     <origin xyz="0 0 0" rpy="0 0 0" />
   </xacro:mrvk_base>
   <!--<xacro:kv01_arm parent="base_end_point" end_point = "tool_point">-->

Commit message: mrvk description: Changed tf in urdf to match position of adis16488.

File: mrvk_description/urdf/mrvk.urdf.xacro (robot description, xacro)
@@ -53,6 +53,11 @@
             </collision>
         </link>
+        <!--Old imu <joint name="stabilizer_to_imu" type="fixed">
+            <origin  xyz="-0.1 0.1 -0.01"/>
+            <parent link="base_stabilized"/>
+            <child link="imu"/>
+        </joint>-->
         <joint name="stabilizer_to_imu" type="fixed">
-            <origin xyz="-0.1 0.1 -0.01"/>
+            <origin rpy = "0 3.14 0" xyz="0.09 0.0 0.625"/>
             <parent link="base_stabilized"/>
             <child link="imu"/>

Commit message: Rozne matejove work in progress veci V pripade potreby revertnut

File: mrvk_description/urdf/mrvk.urdf.xacro (robot description, xacro)
@@ -53,15 +53,16 @@
             </collision>
         </link>
-        <!--Old imu <joint name="stabilizer_to_imu" type="fixed">
-            <origin  xyz="-0.1 0.1 -0.01"/>
-            <parent link="base_stabilized"/>
-            <child link="imu"/>
-        </joint>-->
-        <joint name="stabilizer_to_imu" type="fixed">
+        <joint name="stabilizer_to_adis16350" type="fixed">
+            <origin  xyz="0.0 0.0 -0.01"/>
+            <parent link="base_stabilized"/>
+            <child link="adis16350"/>
+        </joint>
+        <link name = "adis16350"/>
+        <joint name="stabilizer_to_adis16488" type="fixed">
             <origin rpy = "0 3.14 0" xyz="0.09 0.0 0.625"/>
             <parent link="base_stabilized"/>
-            <child link="imu"/>
-        </joint>
-        <link name = "imu"/>
+            <child link="adis16488"/>
+        </joint>
+        <link name = "adis16488"/>
         <link name="laser">
             <visual>
