Commit message: point cloud obstavcle source, adis driver fix

File: mrvk_description/urdf/mrvk.urdf.xacro (robot description, xacro)
@@ -60,5 +60,5 @@
         <link name = "adis16350"/>
         <joint name="stabilizer_to_adis16488" type="fixed">
-            <origin rpy = "0 3.14 0" xyz="0.09 0.0 0.625"/>
+            <origin rpy = "0 0 0" xyz="0.09 0.0 0.625"/>
             <parent link="base_stabilized"/>
             <child link="adis16488"/>

Commit message: Changed robot urdf to reflect new position of ADIS. Added fila with basic commands.

File: mrvk_description/urdf/mrvk.urdf.xacro (robot description, xacro)
@@ -60,5 +60,5 @@
         <link name = "adis16350"/>
         <joint name="stabilizer_to_adis16488" type="fixed">
-            <origin rpy = "0 0 0" xyz="0.09 0.0 0.625"/>
+            <origin rpy = "0 0 ${-M_PI/2}" xyz="0.09 0.0 0.625"/>
             <parent link="base_stabilized"/>
             <child link="adis16488"/>

Commit message: mrvk changes, camera param setup

File: mrvk_description/urdf/mrvk.urdf.xacro (robot description, xacro)
@@ -170,5 +170,11 @@
             <child link="kinect"/>
             <origin rpy=" 0 0.35 0" xyz="0.100 0 0.489"/>
-        </joint>
+            <origin rpy=" 0 0.35 0" xyz="0.110 0 0.65"/>
+        </joint>
+	<!--<joint name="kinect_to_veza" type="fixed">
+            <parent link="base_stabilized"/>
+            <child link="kinect"/>
+            <origin rpy=" 0 0.35 0" xyz="0.100 0 0.489"/>
+        </joint>-->
         <link name="kinect_ir">
         </link>
@@ -176,6 +182,11 @@
             <parent link="kinect"/>
             <child link="kinect_ir"/>
+            <origin rpy="1.57 0 1.57" xyz="0.0 0 0"/>
+        </joint>
+	<!--<joint name="kinect_ir_to_veza" type="fixed">
+            <parent link="kinect"/>
+            <child link="kinect_ir"/>
             <origin rpy="1.57 0 1.57" xyz="0.0 -0.070 0"/>
-        </joint>
+        </joint>-->
         <link name="wheel_frame_l">
             <visual>

Commit message: Adis position update

File: mrvk_description/urdf/mrvk.urdf.xacro (robot description, xacro)
@@ -60,5 +60,5 @@
         <link name = "adis16350"/>
         <joint name="stabilizer_to_adis16488" type="fixed">
-            <origin rpy = "0 0 ${-M_PI/2}" xyz="0.09 0.0 0.625"/>
+            <origin rpy = "0 0 ${-M_PI/2}" xyz="0.0 0.105 0.099"/>
             <parent link="base_stabilized"/>
             <child link="adis16488"/>
