Commit message: xacro fix

File: adis16488/urdf/adis.xacro (robot description, xacro)
@@ -1,8 +1,7 @@
-<?xml version="1.0" ?>
-<robot name="aaa" xmlns:xacro="http://ros.org/wiki/xacro">
-    <xacro:include filename="$(find adis16488)/urdf/afis_frame_macro.xacro"/> <!--Scanner values-->
-    <xacro:Adis parrent = "map">
+<robot name="adis" xmlns:xacro="http://ros.org/wiki/xacro">
+    <xacro:include filename="$(find adis16488)/urdf/adis_frame_macro.xacro"/> <!--Scanner values-->
+    <link name = "map"/>
+    <xacro:Adis parrent ="map">
         <origin xyz="0 0 0" rpy="0 0 0" /> <!--PhoXi3Dscanner origin-->
-    </xacro:PhoXi3Dscanner>
-    <link name ="base_link"/>
+    </xacro:Adis>
 </robot>

File: adis16488/urdf/adis_frame_macro.xacro (robot description, xacro)
@@ -1,11 +1,10 @@
-<?xml version="1.0"?>
 <robot xmlns:xacro="http://ros.org/wiki/xacro">
-    <xacro:macro name = "Adis"
-        <joint name="stabilizer_to_adis16350" type="fixed" params parrent *origin>
+    <xacro:macro name = "Adis" params="parrent *origin">
+        <joint name="adis16350_joint" type="fixed">
             <xacro:insert_block name="origin" />
-            <parent link=${parrent}/>
+            <parent link="${parrent}"/>
             <child link="adis16350"/>
         </joint>
         <link name = "adis16350"/>
       </xacro:macro>
-<robot/>
+</robot>
