Commit message: Model and launch files refactor

File: adis16488/urdf/adis_macro.xacro (robot description, xacro)
@@ -1,10 +1,10 @@
 <robot xmlns:xacro="http://ros.org/wiki/xacro">
-    <xacro:macro name = "Adis" params="parrent *origin">
+    <xacro:macro name = "Adis" params="parent child *origin">
         <joint name="adis16350_joint" type="fixed">
             <xacro:insert_block name="origin" />
-            <parent link="${parrent}"/>
-            <child link="adis16350"/>
+            <parent link="${parent}"/>
+            <child link="${child}"/>
         </joint>
-        <link name = "adis16350"/>
+        <link name = "${child}"/>
       </xacro:macro>
 </robot>

File: mrvk_description/urdf/mrvk.urdf.xacro (robot description, xacro)
@@ -1,4 +1,4 @@
 <?xml version="1.0"?>
-<robot xmlns:xacro="http://www.ros.org/wiki/xacro"
+<robot xmlns:xacro="http://ros.org/wiki/xacro"
        xmlns:xi="http://www.w3.org/2001/XInclude"
        xmlns:gazebo="http://playerstage.sourceforge.net/gazebo/xmlschema/#gz"
@@ -53,16 +53,4 @@
             </collision>
         </link>
-        <joint name="stabilizer_to_adis16350" type="fixed">
-            <origin  xyz="0.0 0.0 -0.01"/>
-            <parent link="base_stabilized"/>
-            <child link="adis16350"/>
-        </joint>
-        <link name = "adis16350"/>
-        <joint name="stabilizer_to_adis16488" type="fixed">
-            <origin rpy = "0 0 ${-M_PI/2}" xyz="0.0 0.105 0.099"/>
-            <parent link="base_stabilized"/>
-            <child link="adis16488"/>
-        </joint>
-        <link name = "adis16488"/>
         <link name="laser">
             <visual>
@@ -154,39 +142,4 @@
             <axis xyz="0 0 1"/>
         </joint>
-        <link name="kinect">
-            <visual>
-                <geometry>
-                    <box size=" .065 0.25 .075"/>
-                </geometry>
-                <material name="kinect"/>
-            </visual>
-            <inertial>
-                <mass value="1.5"/>
-                <inertia_zaklad/>
-            </inertial>
-        </link>
-        <joint name="kinect_to_veza" type="fixed">
-            <parent link="base_stabilized"/>
-            <child link="kinect"/>
-            <origin rpy=" 0 0.35 0" xyz="0.100 0 0.489"/>
-            <origin rpy=" 0 0.35 0" xyz="0.110 0 0.65"/>
-        </joint>
-	<!--<joint name="kinect_to_veza" type="fixed">
-            <parent link="base_stabilized"/>
-            <child link="kinect"/>
-            <origin rpy=" 0 0.35 0" xyz="0.100 0 0.489"/>
-        </joint>-->
-        <link name="kinect_ir">
-        </link>
-        <joint name="kinect_ir_to_veza" type="fixed">
-            <parent link="kinect"/>
-            <child link="kinect_ir"/>
-            <origin rpy="1.57 0 1.57" xyz="0.0 0 0"/>
-        </joint>
-	<!--<joint name="kinect_ir_to_veza" type="fixed">
-            <parent link="kinect"/>
-            <child link="kinect_ir"/>
-            <origin rpy="1.57 0 1.57" xyz="0.0 -0.070 0"/>
-        </joint>-->
         <link name="wheel_frame_l">
             <visual>
@@ -348,16 +301,4 @@
         </joint>
         <link name="${end_point}"/>
-        <joint name="base_to_gps" type="fixed">
-            <parent link="base_link"/>
-            <child link="gps"/>
-            <origin rpy="0 0 0" xyz="0 0 2"/>
-        </joint>
-        <link name="gps"/>
-        <joint name="gps_to_vo" type="fixed">
-            <parent link="gps"/>
-            <child link="vo"/>
-            <origin rpy="0 0 0" xyz="0 0 0"/>
-        </joint>
-        <link name="vo"/>
         <transmission name="mrvk_left_transmission">
             <type>transmission_interface/SimpleTransmission</type>

File: mrvk_sensors/urdf/camera.xacro (robot description, xacro)
@@ -1,7 +1,7 @@
 <robot name="adis" xmlns:xacro="http://ros.org/wiki/xacro">
-    <xacro:include filename="$(find adis16488)/urdf/adis_macro.xacro"/> <!--Scanner values-->
+    <xacro:include filename="$(find mrvk_sensors)/urdf/camera_macro.xacro"/> <!--Scanner values-->
     <link name = "map"/>
-    <xacro:Adis parent ="map" child="adis16488">
+    <xacro:Camera parent ="map" child="camera">
         <origin xyz="0 0 0" rpy="0 0 0" /> <!--PhoXi3Dscanner origin-->
-    </xacro:Adis>
+    </xacro:Camera>
 </robot>

File: mrvk_sensors/urdf/gps.xacro (robot description, xacro)
@@ -1,7 +1,7 @@
 <robot name="adis" xmlns:xacro="http://ros.org/wiki/xacro">
-    <xacro:include filename="$(find adis16488)/urdf/adis_macro.xacro"/> <!--Scanner values-->
+    <xacro:include filename="$(find mrvk_sensors)/urdf/gps_macro.xacro"/> <!--Scanner values-->
     <link name = "map"/>
-    <xacro:Adis parent ="map" child="adis16488">
+    <xacro:Gps parent ="map" chld="gps">
         <origin xyz="0 0 0" rpy="0 0 0" /> <!--PhoXi3Dscanner origin-->
-    </xacro:Adis>
+    </xacro:Gps>
 </robot>

File: mrvk_sensors/urdf/hokuyo.xacro (robot description, xacro)
@@ -1,7 +1,7 @@
 <robot name="adis" xmlns:xacro="http://ros.org/wiki/xacro">
-    <xacro:include filename="$(find adis16488)/urdf/adis_macro.xacro"/> <!--Scanner values-->
+    <xacro:include filename="$(find mrvk_sensors)/urdf/hokuyo_macro.xacro"/> <!--Scanner values-->
     <link name = "map"/>
-    <xacro:Adis parent ="map" child="adis16488">
+    <xacro:Hokuyo parent ="map" child="laser">
         <origin xyz="0 0 0" rpy="0 0 0" /> <!--PhoXi3Dscanner origin-->
-    </xacro:Adis>
+    </xacro:Hokuyo>
 </robot>
