Commit message: robot config

File: mrvk_sensors/urdf/robot.xacro (robot description, xacro)
@@ -30,5 +30,5 @@
     </xacro:mrvk_base>
     <xacro:Adis parent="base_stabilized" child = "adis16488">
-        <origin rpy = "0 0 ${-M_PI/2}" xyz="0.0 0.105 0.099"/>
+        <origin rpy = "0 0 0" xyz="0.0 0.0 0.099"/>
     </xacro:Adis>
     <xacro:Gps parent="base_stabilized" child = "gps">

Commit message: Fix camera frame refaktor, filter cloud

File: mrvk_sensors/urdf/robot.xacro (robot description, xacro)
@@ -36,5 +36,5 @@
     </xacro:Gps>
     <xacro:Camera parent="base_stabilized" child = "camera_frame">
-        <origin rpy="1.57 0 1.57" xyz="0.1 -0.070 0.489"/>
+        <origin rpy="1.80 0 1.57" xyz="0.1 -0.070 0.489"/> <!-- 1.57 0 1.57 -->
     </xacro:Camera>
     <!--<xacro:Hokuyo parent="base_stabilized" child = "laser">-->
